File: Main.sch (KiCad schematic (older format))
At the start: 60 parts, among them J1 Conn_02x06_Top_Bottom, J6 Conn_01x03, J7 Conn_01x03, J8 Conn_01x06, Q1 CSD17307Q5A, Q2 CSD17307Q5A, U1 LM4120-CustomSymbols, U2 LTC2942, U3 LM393, U4 TPS2557, U5 LM393, U6 TPS2557, U7 SN74LVC2G08

Commit message: restarted
Parts:
- removed AL/CC1, BAT+1, BAT-1, PACK+1, SCL1, SDA1: TestPoint, Connector_PinHeader_2.00mm:PinHeader_1x01_P2.00mm_Vertical, symbol Connector:TestPoint
- added J2: Conn_01x06_Male, Connector_PinSocket_2.00mm:PinSocket_1x06_P2.00mm_Vertical, symbol Connector:Conn_01x06_Male
Connections:
- net BAT+1: now reaches BT1.1 (+), C2.1, R16.2, R7.1, SHORT1.1, U2.1 (SENSE+)
- net BAT+1: now also J2.1 (Pin_1)
- net PACK+1: now reaches OUT1.1, R16.1, U2.6 (SENSE-)
- net PACK+1: now also J2.6 (Pin_6)
- net SCL1: now reaches U2.3 (SCL)
- net SCL1: now also J2.3 (Pin_3)
- net SDA1: now reaches U2.4 (SDA)
- net SDA1: now also J2.4 (Pin_4)
- net AL_CC1: now reaches U2.5 (AL/CC)
- net AL_CC1: now also J2.5 (Pin_5)
- net BQ29707_P4 renamed BAT-1
- net BAT-1: now also J2.2 (Pin_2)
Changed lines of the file:
@@
-$EndComp
-$Comp
-L Connector:TestPoint SCL1
-U 1 1 5DE9DE05
-P 6900 9450
-F 0 "SCL1" V 6800 9600 50  0000 C CNN
-F 1 "TestPoint" V 6700 9600 50  0000 C CNN
-F 2 "Connector_PinHeader_2.00mm:PinHeader_1x01_P2.00mm_Vertical" H 7100 9450 50  0001 C CNN
-F 3 "~" H 7100 9450 50  0001 C CNN
-	1    6900 9450
-	0    -1   -1   0
-$EndComp
-$Comp
-L Connector:TestPoint SDA1
-U 1 1 5DE9F47E
-P 7900 9450
-F 0 "SDA1" V 7854 9638 50  0000 L CNN
-F 1 "TestPoint" V 7945 9638 50  0000 L CNN
-F 2 "Connector_PinHeader_2.00mm:PinHeader_1x01_P2.00mm_Vertical" H 8100 9450 50  0001 C CNN
-F 3 "~" H 8100 9450 50  0001 C CNN
-	1    7900 9450
-	0    1    1    0
-$EndComp
-$Comp
-L Connector:TestPoint AL/CC1
-U 1 1 5DE9FAC6
-P 7900 9150
-F 0 "AL/CC1" V 7854 9338 50  0000 L CNN
-F 1 "TestPoint" V 7945 9338 50  0000 L CNN
-F 2 "Connector_PinHeader_2.00mm:PinHeader_1x01_P2.00mm_Vertical" H 8100 9150 50  0001 C CNN
-F 3 "~" H 8100 9150 50  0001 C CNN
-	1    7900 9150
-	0    1    1    0
 $EndComp
 $Comp
@@
 Wire Wire Line
 	5650 6450 5650 6350
-$Comp
-L Connector:TestPoint PACK+1
-U 1 1 5E5B47FA
-P 8450 7850
-F 0 "PACK+1" H 8508 7968 50  0000 L CNN
-F 1 "TestPoint" H 8508 7877 50  0000 L CNN
-F 2 "Connector_PinHeader_2.00mm:PinHeader_1x01_P2.00mm_Vertical" H 8650 7850 50  0001 C CNN
-F 3 "~" H 8650 7850 50  0001 C CNN
-	1    8450 7850
-	1    0    0    -1
-$EndComp
-Wire Wire Line
-	8450 8350 8450 7850
 Wire Wire Line
 	8450 8350 8450 8900
 Wire Wire Line
 	4800 8000 4800 8350
-$Comp
-L Connector:TestPoint BAT+1
-U 1 1 5E5C1DD0
-P 4800 8000
-F 0 "BAT+1" H 4858 8118 50  0000 L CNN
-F 1 "TestPoint" H 4858 8027 50  0000 L CNN
-F 2 "Connector_PinHeader_2.00mm:PinHeader_1x01_P2.00mm_Vertical" H 5000 8000 50  0001 C CNN
-F 3 "~" H 5000 8000 50  0001 C CNN
-	1    4800 8000
-	1    0    0    -1
-$EndComp
-Wire Wire Line
-	4800 9300 4800 9600
-Connection ~ 4800 9300
-$Comp
-L Connector:TestPoint BAT-1
-U 1 1 5E5C8259
-P 4800 9600
-F 0 "BAT-1" H 4742 9626 50  0000 R CNN
-F 1 "TestPoint" H 4742 9717 50  0000 R CNN
-F 2 "Connector_PinHeader_2.00mm:PinHeader_1x01_P2.00mm_Vertical" H 5000 9600 50  0001 C CNN
-F 3 "~" H 5000 9600 50  0001 C CNN
-	1    4800 9600
-	-1   0    0    1
-$EndComp
 Wire Wire Line
 	14750 8350 14750 8000
@@
 Text Notes 9750 4150 0    50   ~ 0
 Comparator Supply Bypass Capacitor
+$Comp
+L Connector:Conn_01x06_Male J2
+U 1 1 5DFA344A
+P 7200 10650
+F 0 "J2" V 7262 10894 50  0000 L CNN
+F 1 "Conn_01x06_Male" V 7353 10894 50  0000 L CNN
+F 2 "Connector_PinSocket_2.00mm:PinSocket_1x06_P2.00mm_Vertical" H 7200 10650 50  0001 C CNN
+F 3 "~" H 7200 10650 50  0001 C CNN
+	1    7200 10650
+	0    -1   -1   0
+$EndComp
+Text GLabel 7000 10450 1    50   Input ~ 0
+BAT+1
+Text GLabel 7100 10450 1    50   Input ~ 0
+BAT-1
+Text GLabel 4800 8000 1    50   Input ~ 0
+BAT+1
+Text GLabel 4800 9400 3    50   Input ~ 0
+BAT-1
+Wire Wire Line
+	4800 9300 4800 9400
+Connection ~ 4800 9300
+Text GLabel 7200 10450 1    50   Input ~ 0
+SCL1
+Text GLabel 6900 9450 0    50   Input ~ 0
+SCL1
+Text GLabel 7300 10450 1    50   Input ~ 0
+SDA1
+Text GLabel 7900 9450 2    50   Input ~ 0
+SDA1
+Text GLabel 7900 9150 2    50   Input ~ 0
+AL_CC1
+Text GLabel 7400 10450 1    50   Input ~ 0
+AL_CC1
+Text GLabel 7500 10450 1    50   Input ~ 0
+PACK+1
+Wire Wire Line
+	8450 8350 8450 8200
+Text GLabel 8450 8200 1    50   Input ~ 0
+PACK+1
 $EndSCHEMATC

Commit message: changed test points
Parts:
- removed J1: Conn_02x06_Top_Bottom, Connector_PinHeader_2.00mm:PinHeader_2x06_P2.00mm_Vertical, symbol Connector_Generic:Conn_02x06_Top_Bottom
- added C10: 0.1u, Capacitor_SMD:C_1206_3216Metric_Pad1.42x1.75mm_HandSolder, symbol Device:C
- added J1, J4: Conn_01x01_Male, Connector_PinHeader_2.00mm:PinHeader_1x01_P2.00mm_Vertical, symbol Connector:Conn_01x01_Male
- added J3, J5: Conn_01x05_Male, Connector_PinHeader_2.00mm:PinHeader_1x05_P2.00mm_Vertical, symbol Connector:Conn_01x05_Male
- added J9: Conn_01x06_Male, Connector_PinHeader_2.00mm:PinHeader_1x06_P2.00mm_Vertical, symbol Connector:Conn_01x06_Male
Connections:
- net 1.4Vref: now also J5.3 (Pin_3)
- net 5Vref: now also J1.1 (Pin_1)
- net 933mVref: now also J5.4 (Pin_4)
- net BATdiv3: now also J5.2 (Pin_2)
- net BatTemp: now also J3.1 (Pin_1), J3.3 (Pin_3)
- net ChargeEnable: now also J9.3 (Pin_3)
- net ChargeOK: now also J5.1 (Pin_1), J9.5 (Pin_5)
- net DischargeEnable: now also J9.6 (Pin_6)
- net DischargeOK: now also J5.5 (Pin_5), J9.1 (Pin_1)
- net GNDA: now also C10.2
- net HighTemp: now also J3.2 (Pin_2)
- net LowTemp: now also J3.4 (Pin_4)
- net PACK+: now also C10.1, J4.1 (Pin_1)
- net TempOK: now also J3.5 (Pin_5), J9.2 (Pin_2), J9.4 (Pin_4)
Other:
- note added: "AND GATE Supply Bypass Capacitor"
- note added: "BQ29707 Test Points"
- note removed: "Silk screen will be used to label all the TP's\n\n"
- moved on the sheet: BT1, C1, C2, C3, C4, C5, C6, C7, C8, C9, CDR1, D1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
