File: Main.sch (KiCad schematic (older format))
At the start: 60 parts, among them J1 Conn_01x01_Male, J2 Conn_01x06_Male, J3 Conn_01x05_Male, J4 Conn_01x01_Male, J5 Conn_01x05_Male, J6 Conn_01x03, J7 Conn_01x03, J8 Conn_01x06, J9 Conn_01x06_Male, Q1 CSD17307Q5A, Q2 CSD17307Q5A, U1 LM4120-CustomSymbols, U2 LTC2942, U3 LM393, U4 TPS2557, U5 LM393, U6 TPS2557, U7 SN74LVC2G08

Commit message: progress
Other:
- note added: "Battery Control"
- note added: "Battery Protection, Columb Counter and Charging/Discharge Load switches"
- moved on the sheet: BT1, C1, C2, C3, C4, C5, C6, C7, C8, CDR1, GND1, J1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

Commit message: progress
Other:
- note added: "Battery Protection, Columb Counter and Discharge/Charge Load switches"
- note removed: "Battery Protection, Columb Counter and Charging/Discharge Load switches"
Changed lines of the file:
@@
 Battery Control
 Text Notes 3550 4750 0    157  ~ 0
-Battery Protection, Columb Counter and Charging/Discharge Load switches
+Battery Protection, Columb Counter and Discharge/Charge Load switches
 $EndSCHEMATC

Commit message: progress
Other:
- note added: "Battery Protection, Coloumb Counter and Discharge/Charge Load switches"
- note removed: "Battery Protection, Columb Counter and Discharge/Charge Load switches"
Changed lines of the file:
@@
 Battery Control
 Text Notes 3550 4750 0    157  ~ 0
-Battery Protection, Columb Counter and Discharge/Charge Load switches
+Battery Protection, Coloumb Counter and Discharge/Charge Load switches
 $EndSCHEMATC
