File: Main.sch (KiCad schematic (older format))
At the start: 60 parts, among them J1 Conn_01x01_Male, J2 Conn_01x06_Male, J3 Conn_01x05_Male, J4 Conn_01x01_Male, J5 Conn_01x05_Male, J6 Conn_01x03, J7 Conn_01x03, J8 Conn_01x06, J9 Conn_01x06_Male, Q1 CSD17307Q5A, Q2 CSD17307Q5A, U1 LM4120-CustomSymbols, U2 LTC2942, U3 LM393, U4 TPS2557, U5 LM393, U6 TPS2557, U7 SN74LVC2G08

Commit message: removed_switches
Parts:
- removed OUT1, SHORT1: SW_Push, Button_Switch_SMD:SW_DIP_SPSTx01_Slide_6.7x4.1mm_W6.73mm_P2.54mm_LowProfile_JPin, symbol Switch:SW_Push
- added JP1, JP2: Jumper_2_Open, Connector_PinHeader_2.00mm:PinHeader_1x02_P2.00mm_Vertical, symbol Jumper:Jumper_2_Open
Changed lines of the file:
@@
 Wire Wire Line
 	8900 7750 8700 7750
-$Comp
-L Switch:SW_Push OUT1
-U 1 1 5E2FB6C9
-P 9100 7750
-F 0 "OUT1" H 9000 8100 50  0000 L CNN
-F 1 "SW_Push" H 9000 8000 50  0000 L CNN
-F 2 "Button_Switch_SMD:SW_DIP_SPSTx01_Slide_6.7x4.1mm_W6.73mm_P2.54mm_LowProfile_JPin" H 9100 7950 50  0001 C CNN
-F 3 "~" H 9100 7950 50  0001 C CNN
-	1    9100 7750
-	1    0    0    -1
-$EndComp
 Wire Wire Line
 	7850 7750 8700 7750
@@
 Wire Wire Line
 	5800 8100 5800 7750
-$Comp
-L Switch:SW_Push SHORT1
-U 1 1 5D0F6604
-P 5800 8300
-F 0 "SHORT1" V 5754 8448 50  0000 L CNN
-F 1 "SW_Push" V 5845 8448 50  0000 L CNN
-F 2 "Button_Switch_SMD:SW_DIP_SPSTx01_Slide_6.7x4.1mm_W6.73mm_P2.54mm_LowProfile_JPin" H 5800 8500 50  0001 C CNN
-F 3 "~" H 5800 8500 50  0001 C CNN
-	1    5800 8300
-	0    1    1    0
-$EndComp
 Wire Wire Line
 	3150 8300 3150 8400
@@
 Wire Notes Line
 	1000 5000 1000 1100
+$Comp
+L Jumper:Jumper_2_Open JP2
+U 1 1 5DF47769
+P 9100 7750
+F 0 "JP2" H 9100 7525 50  0000 C CNN
+F 1 "Jumper_2_Open" H 9100 7600 50  0000 C CNN
+F 2 "Connector_PinHeader_2.00mm:PinHeader_1x02_P2.00mm_Vertical" H 9100 7750 50  0001 C CNN
+F 3 "~" H 9100 7750 50  0001 C CNN
+	1    9100 7750
+	1    0    0    -1
+$EndComp
+$Comp
+L Jumper:Jumper_2_Open JP1
+U 1 1 5DF5F15C
+P 5800 8300
+F 0 "JP1" H 5800 8075 50  0000 C CNN
+F 1 "Jumper_2_Open" H 5800 8150 50  0000 C CNN
+F 2 "Connector_PinHeader_2.00mm:PinHeader_1x02_P2.00mm_Vertical" H 5800 8300 50  0001 C CNN
+F 3 "~" H 5800 8300 50  0001 C CNN
+	1    5800 8300
+	0    -1   -1   0
+$EndComp
 $EndSCHEMATC

Commit message: progress
Parts:
- JP1, JP2: footprint Connector_PinHeader_2.00mm:PinHeader_1x02_P2.00mm_Vertical -> Connector_PinSocket_2.54mm:PinSocket_1x01_P2.54mm_Vertical
Changed lines of the file:
@@
 F 0 "JP2" H 9100 7525 50  0000 C CNN
 F 1 "Jumper_2_Open" H 9100 7600 50  0000 C CNN
-F 2 "Connector_PinHeader_2.00mm:PinHeader_1x02_P2.00mm_Vertical" H 9100 7750 50  0001 C CNN
+F 2 "Connector_PinSocket_2.54mm:PinSocket_1x01_P2.54mm_Vertical" H 9100 7750 50  0001 C CNN
 F 3 "~" H 9100 7750 50  0001 C CNN
 	1    9100 7750
@@
 F 0 "JP1" H 5800 8075 50  0000 C CNN
 F 1 "Jumper_2_Open" H 5800 8150 50  0000 C CNN
-F 2 "Connector_PinHeader_2.00mm:PinHeader_1x02_P2.00mm_Vertical" H 5800 8300 50  0001 C CNN
+F 2 "Connector_PinSocket_2.54mm:PinSocket_1x01_P2.54mm_Vertical" H 5800 8300 50  0001 C CNN
 F 3 "~" H 5800 8300 50  0001 C CNN
 	1    5800 8300

Commit message: progress
Parts:
- removed J3: Conn_01x05_Male, Connector_PinHeader_2.00mm:PinHeader_1x05_P2.00mm_Vertical, symbol Connector:Conn_01x05_Male
- removed J9: Conn_01x06_Male, Connector_PinHeader_2.00mm:PinHeader_1x06_P2.00mm_Vertical, symbol Connector:Conn_01x06_Male
- added J3: Conn_01x04_Male, Connector_PinHeader_2.00mm:PinHeader_1x04_P2.00mm_Vertical, symbol Connector:Conn_01x04_Male
- added J9: Conn_01x05_Male, Connector_PinHeader_2.00mm:PinHeader_1x05_P2.00mm_Vertical, symbol Connector:Conn_01x05_Male
Connections:
- net BatTemp: now also J3.1 (Pin_1)
- net ChargeEnable: now also J9.3 (Pin_3)
- net ChargeOK: now also J9.4 (Pin_4)
- net DischargeEnable: now also J9.5 (Pin_5)
- net DischargeOK: now also J9.1 (Pin_1)
- net HighTemp: now also J3.2 (Pin_2)
- net LowTemp: now also J3.3 (Pin_3)
- net TempOK: now also J3.4 (Pin_4), J9.2 (Pin_2)
Changed lines of the file:
@@
 	0    -1   -1   0
 $EndComp
-$Comp
-L Connector:Conn_01x05_Male J3
-U 1 1 5DFA2C02
-P 8350 3150
-F 0 "J3" V 8504 2862 50  0000 R CNN
-F 1 "Conn_01x05_Male" V 8413 2862 50  0000 R CNN
-F 2 "Connector_PinHeader_2.00mm:PinHeader_1x05_P2.00mm_Vertical" H 8350 3150 50  0001 C CNN
-F 3 "~" H 8350 3150 50  0001 C CNN
-	1    8350 3150
-	0    -1   -1   0
-$EndComp
-Text GLabel 8150 2950 1    50   Input ~ 0
+Text GLabel 8150 2800 1    50   Input ~ 0
 BatTemp
-Text GLabel 8250 2950 1    50   Input ~ 0
+Text GLabel 8250 2800 1    50   Input ~ 0
 HighTemp
-Text GLabel 8350 2950 1    50   Input ~ 0
-BatTemp
-Text GLabel 8450 2950 1    50   Input ~ 0
+Text GLabel 8350 2800 1    50   Input ~ 0
 LowTemp
-Text GLabel 8550 2950 1    50   Input ~ 0
+Text GLabel 8450 2800 1    50   Input ~ 0
 TempOK
-Text GLabel 14300 3150 1    50   Input ~ 0
+Text GLabel 14400 3050 1    50   Input ~ 0
+ChargeOK
+Text GLabel 14500 3050 1    50   Input ~ 0
+DischargeEnable
+Text GLabel 14300 3050 1    50   Input ~ 0
+ChargeEnable
+Text GLabel 14200 3050 1    50   Input ~ 0
 TempOK
-Text GLabel 14400 3150 1    50   Input ~ 0
-ChargeOK
-Text GLabel 14500 3150 1    50   Input ~ 0
-DischargeEnable
-Text GLabel 14200 3150 1    50   Input ~ 0
-ChargeEnable
-Text GLabel 14100 3150 1    50   Input ~ 0
-TempOK
-Text GLabel 14000 3150 1    50   Input ~ 0
+Text GLabel 14100 3050 1    50   Input ~ 0
 DischargeOK
-$Comp
-L Connector:Conn_01x06_Male J9
-U 1 1 5DFC1AB1
-P 14200 3350
-F 0 "J9" V 14354 2962 50  0000 R CNN
-F 1 "Conn_01x06_Male" V 14263 2962 50  0000 R CNN
-F 2 "Connector_PinHeader_2.00mm:PinHeader_1x06_P2.00mm_Vertical" H 14200 3350 50  0001 C CNN
-F 3 "~" H 14200 3350 50  0001 C CNN
-	1    14200 3350
-	0    -1   -1   0
-$EndComp
 $Comp
 L Main-rescue:SN74LVC2G08-CustomSymbols U7
@@
 Wire Notes Line
 	1000 1100 15450 1100
-Wire Notes Line
-	15450 1100 15450 5000
 Text Notes 7250 1000 0    157  ~ 0
 Battery Control
@@
 	0    -1   -1   0
 $EndComp
+$Comp
+L Connector:Conn_01x04_Male J3
+U 1 1 5DF9ED68
+P 8250 3000
+F 0 "J3" V 8404 2712 50  0000 R CNN
+F 1 "Conn_01x04_Male" V 8313 2712 50  0000 R CNN
+F 2 "Connector_PinHeader_2.00mm:PinHeader_1x04_P2.00mm_Vertical" H 8250 3000 50  0001 C CNN
+F 3 "~" H 8250 3000 50  0001 C CNN
+	1    8250 3000
+	0    -1   -1   0
+$EndComp
+$Comp
+L Connector:Conn_01x05_Male J9
+U 1 1 5E03D4C2
+P 14300 3250
+F 0 "J9" V 14454 2962 50  0000 R CNN
+F 1 "Conn_01x05_Male" V 14363 2962 50  0000 R CNN
+F 2 "Connector_PinHeader_2.00mm:PinHeader_1x05_P2.00mm_Vertical" H 14300 3250 50  0001 C CNN
+F 3 "~" H 14300 3250 50  0001 C CNN
+	1    14300 3250
+	0    -1   -1   0
+$EndComp

Commit message: progress
Changed lines of the file:
@@
 Wire Wire Line
 	13750 4400 13750 4300
-$Comp
-L power:GNDD #PWR023
-U 1 1 5E551E1B
-P 13750 4400
-F 0 "#PWR023" H 13750 4150 50  0001 C CNN
-F 1 "GNDD" H 13754 4245 50  0000 C CNN
-F 2 "" H 13750 4400 50  0001 C CNN
-F 3 "" H 13750 4400 50  0001 C CNN
-	1    13750 4400
-	1    0    0    -1
-$EndComp
 Text GLabel 13850 4100 0    50   Input ~ 0
 ChargeEnable
@@
 	0    -1   -1   0
 $EndComp
+Wire Notes Line
+	15450 5000 15450 1100
+$Comp
+L power:GNDD #PWR?
+U 1 1 5E111712
+P 13750 4400
+F 0 "#PWR?" H 13750 4150 50  0001 C CNN
+F 1 "GNDD" H 13754 4245 50  0000 C CNN
+F 2 "" H 13750 4400 50  0001 C CNN
+F 3 "" H 13750 4400 50  0001 C CNN
+	1    13750 4400
+	1    0    0    -1
+$EndComp
 $EndSCHEMATC

Commit message: done
Connections:
- net GNDD is gone; now on net GNDA: C1.2, C2.2, C4.2, C5.2, C6.2, C7.2, C8.2, GND1.1, JP1.1 (A), Q1.1 (S), Q1.2 (S), Q1.3 (S), R20.2, R21.2, R3.1, R4.1, U1.2 (GND), U2.2 (GND), U4.1 (GND), U6.1 (GND), U7.4 (GND)
Changed lines of the file:
@@
 	1    0    0    -1
 $EndComp
+$Comp
+L power:GNDD #PWR?
+U 1 1 5DF8B5AD
+P 1450 1450
+F 0 "#PWR?" H 1450 1200 50  0001 C CNN
+F 1 "GNDD" H 1454 1295 50  0000 C CNN
+F 2 "" H 1450 1450 50  0001 C CNN
+F 3 "" H 1450 1450 50  0001 C CNN
+	1    1450 1450
+	1    0    0    -1
+$EndComp
+$Comp
+L power:GNDA #PWR?
+U 1 1 5DF92BD0
+P 1750 1450
+F 0 "#PWR?" H 1750 1200 50  0001 C CNN
+F 1 "GNDA" H 1755 1277 50  0000 C CNN
+F 2 "" H 1750 1450 50  0001 C CNN
+F 3 "" H 1750 1450 50  0001 C CNN
+	1    1750 1450
+	1    0    0    -1
+$EndComp
+Wire Wire Line
+	1450 1450 1450 1300
+Wire Wire Line
+	1450 1300 1750 1300
+Wire Wire Line
+	1750 1300 1750 1450
 $EndSCHEMATC

Commit message: done
Parts:
- removed D1, D2: D_Schottky, Diode_SMD:D_2114_3652Metric_Castellated, symbol Device:D_Schottky
- added D1, D2: DB2431200L, DB2431200L:DB2431200L, symbol DB2431200L:DB2431200L
Connections:
- net MPB: now also D2.1
- net PACK+: now also D1.1
- net at C6.1, CDR1.1, U4.6 (OUT)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: now also D1.2, D2.2
Changed lines of the file:
@@
 	14550 7750 15000 7750
 Connection ~ 14550 7750
-$Comp
-L Device:D_Schottky D1
-U 1 1 5E2A87DC
-P 10850 6750
-F 0 "D1" H 10850 6966 50  0000 C CNN
-F 1 "D_Schottky" H 10850 6875 50  0000 C CNN
-F 2 "Diode_SMD:D_2114_3652Metric_Castellated" H 10850 6750 50  0001 C CNN
-F 3 "~" H 10850 6750 50  0001 C CNN
-	1    10850 6750
-	1    0    0    -1
-$EndComp
-$Comp
-L Device:D_Schottky D2
-U 1 1 5E2A9DAF
-P 13100 6750
-F 0 "D2" H 13100 6534 50  0000 C CNN
-F 1 "D_Schottky" H 13100 6625 50  0000 C CNN
-F 2 "Diode_SMD:D_2114_3652Metric_Castellated" H 13100 6750 50  0001 C CNN
-F 3 "~" H 13100 6750 50  0001 C CNN
-	1    13100 6750
-	-1   0    0    1
-$EndComp
-Wire Wire Line
-	12000 6750 11000 6750
 Wire Wire Line
 	12000 6750 12000 7750
-Wire Wire Line
-	12000 6750 12950 6750
 Connection ~ 12000 6750
 Wire Wire Line
 	9600 7750 9600 6750
-Wire Wire Line
-	13250 6750 14550 6750
 Wire Wire Line
 	14550 6750 14550 7750
@@
 Wire Notes Line
 	9950 2300 9950 5000
-Wire Wire Line
-	9600 6750 10700 6750
 Wire Notes Line
 	7350 5000 7350 2300
@@
 	15450 5000 15450 1100
 $Comp
-L power:GNDD #PWR?
+L power:GNDD #PWR0102
 U 1 1 5E111712
 P 13750 4400
-F 0 "#PWR?" H 13750 4150 50  0001 C CNN
+F 0 "#PWR0102" H 13750 4150 50  0001 C CNN
 F 1 "GNDD" H 13754 4245 50  0000 C CNN
 F 2 "" H 13750 4400 50  0001 C CNN
@@
 $EndComp
 $Comp
-L power:GNDD #PWR?
+L power:GNDD #PWR0103
 U 1 1 5DF8B5AD
 P 1450 1450
-F 0 "#PWR?" H 1450 1200 50  0001 C CNN
+F 0 "#PWR0103" H 1450 1200 50  0001 C CNN
 F 1 "GNDD" H 1454 1295 50  0000 C CNN
 F 2 "" H 1450 1450 50  0001 C CNN
@@
 $EndComp
 $Comp
-L power:GNDA #PWR?
+L power:GNDA #PWR0104
 U 1 1 5DF92BD0
 P 1750 1450
-F 0 "#PWR?" H 1750 1200 50  0001 C CNN
+F 0 "#PWR0104" H 1750 1200 50  0001 C CNN
 F 1 "GNDA" H 1755 1277 50  0000 C CNN
 F 2 "" H 1750 1450 50  0001 C CNN
@@
 Wire Wire Line
 	1750 1300 1750 1450
+Wire Wire Line
+	12000 6750 11200 6750
+Wire Wire Line
+	10450 6750 9600 6750
+Wire Wire Line
+	12000 6750 12850 6750
+Wire Wire Line
+	13600 6750 14550 6750
+$Comp
+L DB2431200L:DB2431200L D1
+U 1 1 5E000D7A
+P 10850 6750
+F 0 "D1" H 10875 6435 50  0000 C CNN
+F 1 "DB2431200L" H 10875 6526 50  0000 C CNN
+F 2 "DB2431200L:DB2431200L" H 11000 7350 50  0001 C CNN
+F 3 "" H 11000 7350 50  0001 C CNN
+	1    10850 6750
+	-1   0    0    1
+$EndComp
+$Comp
+L DB2431200L:DB2431200L D2
+U 1 1 5E001BEF
+P 13200 6750
+F 0 "D2" H 13225 7065 50  0000 C CNN
+F 1 "DB2431200L" H 13225 6974 50  0000 C CNN
+F 2 "DB2431200L:DB2431200L" H 13350 7350 50  0001 C CNN
+F 3 "" H 13350 7350 50  0001 C CNN
+	1    13200 6750
+	1    0    0    -1
+$EndComp
 $EndSCHEMATC

Commit message: changed_footprings
Parts:
- R14: footprint Resistor_SMD:R_1206_3216Metric_Pad1.42x1.75mm_HandSolder -> Resistor_SMD:R_0805_2012Metric_Pad1.15x1.40mm_HandSolder
- R17: footprint Resistor_SMD:R_1206_3216Metric_Pad1.42x1.75mm_HandSolder -> Resistor_SMD:R_0603_1608Metric_Pad1.05x0.95mm_HandSolder
Changed lines of the file:
@@
 F 0 "R14" H 5820 3846 50  0000 L CNN
 F 1 "1.43M" H 5820 3755 50  0000 L CNN
-F 2 "Resistor_SMD:R_1206_3216Metric_Pad1.42x1.75mm_HandSolder" V 5680 3800 50  0001 C CNN
+F 2 "Resistor_SMD:R_0805_2012Metric_Pad1.15x1.40mm_HandSolder" V 5680 3800 50  0001 C CNN
 F 3 "~" H 5750 3800 50  0001 C CNN
 	1    5750 3800
@@
 F 0 "R17" H 9370 3946 50  0000 L CNN
 F 1 "284k" H 9370 3855 50  0000 L CNN
-F 2 "Resistor_SMD:R_1206_3216Metric_Pad1.42x1.75mm_HandSolder" V 9230 3900 50  0001 C CNN
+F 2 "Resistor_SMD:R_0603_1608Metric_Pad1.05x0.95mm_HandSolder" V 9230 3900 50  0001 C CNN
 F 3 "~" H 9300 3900 50  0001 C CNN
 	1    9300 3900

Commit message: progress
Parts:
- added R24: 187k, Resistor_SMD:R_1206_3216Metric_Pad1.42x1.75mm_HandSolder, symbol Device:R
- R1, R2, R8: value 898k -> 887k
- R10: value 332k -> 187k
- R11: value 167k -> 187k
- R12: value 1.64M -> 1.62M
- R16: value 14.7m -> 14m; footprint Resistor_SMD:R_1206_3216Metric_Pad1.42x1.75mm_HandSolder -> Resistor_SMD:R_0805_2012Metric
- U7: footprint Package_SO:SSOP-8_2.95x2.8mm_P0.65mm -> SN74LVC2G08DCTR:SN74LVC2G08DCTR
Connections:
- net BATdiv3: now also R24.2; no longer R10.2
- new net: R10.2, R24.1
Other:
- note added: "BQ29709 Test Points"
- note removed: "BQ29707 Test Points"
Changed lines of the file:
@@
 Text Notes 5000 3400 0    50   ~ 0
 2.5uA
-Text Notes 4350 3400 0    50   ~ 0
+Text Notes 4350 3100 0    50   ~ 0
 5uA
 Text GLabel 5750 3500 2    50   Input ~ 0
@@
 P 5000 3800
 F 0 "R12" H 5070 3846 50  0000 L CNN
-F 1 "1.64M" H 5070 3755 50  0000 L CNN
+F 1 "1.62M" H 5070 3755 50  0000 L CNN
 F 2 "Resistor_SMD:R_1206_3216Metric_Pad1.42x1.75mm_HandSolder" V 4930 3800 50  0001 C CNN
 F 3 "~" H 5000 3800 50  0001 C CNN
@@
 BATdiv3
 Wire Wire Line
-	4300 3650 4300 3500
+	4300 3350 4300 3200
 Wire Wire Line
 	4300 3950 4300 4150
@@
 P 4300 4300
 F 0 "R11" H 4370 4346 50  0000 L CNN
-F 1 "167k" H 4370 4255 50  0000 L CNN
+F 1 "187k" H 4370 4255 50  0000 L CNN
 F 2 "Resistor_SMD:R_1206_3216Metric_Pad1.42x1.75mm_HandSolder" V 4230 4300 50  0001 C CNN
 F 3 "~" H 4300 4300 50  0001 C CNN
 	1    4300 4300
-	1    0    0    -1
-$EndComp
-$Comp
-L Device:R R10
-U 1 1 5E430D59
-P 4300 3800
-F 0 "R10" H 4370 3846 50  0000 L CNN
-F 1 "332k" H 4370 3755 50  0000 L CNN
-F 2 "Resistor_SMD:R_1206_3216Metric_Pad1.42x1.75mm_HandSolder" V 4230 3800 50  0001 C CNN
-F 3 "~" H 4300 3800 50  0001 C CNN
-	1    4300 3800
 	1    0    0    -1
 $EndComp
@@
 P 2800 3800
 F 0 "R2" H 2870 3846 50  0000 L CNN
-F 1 "898k" H 2870 3755 50  0000 L CNN
+F 1 "887k" H 2870 3755 50  0000 L CNN
 F 2 "Resistor_SMD:R_1206_3216Metric_Pad1.42x1.75mm_HandSolder" V 2730 3800 50  0001 C CNN
 F 3 "~" H 2800 3800 50  0001 C CNN
@@
 P 3550 3800
 F 0 "R8" H 3620 3846 50  0000 L CNN
-F 1 "898k" H 3620 3755 50  0000 L CNN
+F 1 "887k" H 3620 3755 50  0000 L CNN
 F 2 "Resistor_SMD:R_1206_3216Metric_Pad1.42x1.75mm_HandSolder" V 3480 3800 50  0001 C CNN
 F 3 "~" H 3550 3800 50  0001 C CNN
@@
 P 2150 3800
 F 0 "R1" H 2220 3846 50  0000 L CNN
-F 1 "898k" H 2220 3755 50  0000 L CNN
+F 1 "887k" H 2220 3755 50  0000 L CNN
 F 2 "Resistor_SMD:R_1206_3216Metric_Pad1.42x1.75mm_HandSolder" V 2080 3800 50  0001 C CNN
 F 3 "~" H 2150 3800 50  0001 C CNN
@@
 Text Notes 1600 4900 0    50   ~ 0
 NTCG Series Thermistor
-Text GLabel 4300 3500 2    50   Input ~ 0
+Text GLabel 4300 3200 2    50   Input ~ 0
 PACK+
 $Comp
@@
 F 0 "U7" H 14275 4565 50  0000 C CNN
 F 1 "SN74LVC2G08" H 14275 4474 50  0000 C CNN
-F 2 "Package_SO:SSOP-8_2.95x2.8mm_P0.65mm" H 14300 4000 50  0001 C CNN
+F 2 "SN74LVC2G08DCTR:SN74LVC2G08DCTR" H 14300 4000 50  0001 C CNN
 F 3 "" H 14300 4000 50  0001 C CNN
 	1    14300 4000
@@
 $EndComp
 Text Notes 1050 7050 0    50   ~ 0
-BQ29707 Test Points
+BQ29709 Test Points
 Text GLabel 8700 7600 1    50   Input ~ 0
 PACK+1
@@
 AR Path="/5D0BC9BA/5DE9CAD1" Ref="R?"  Part="1"
 F 0 "R16" V 7500 7800 50  0000 C CNN
-F 1 "14.7m" V 7600 7750 50  0000 C CNN
-F 2 "Resistor_SMD:R_1206_3216Metric_Pad1.42x1.75mm_HandSolder" V 7630 7750 50  0001 C CNN
+F 1 "14m" V 7600 7750 50  0000 C CNN
+F 2 "Resistor_SMD:R_0805_2012Metric" V 7630 7750 50  0001 C CNN
 F 3 "~" H 7700 7750 50  0001 C CNN
 	1    7700 7750
@@
 	1    0    0    -1
 $EndComp
+$Comp
+L Device:R R24
+U 1 1 5DFA0A4B
+P 4300 3800
+F 0 "R24" H 4370 3846 50  0000 L CNN
+F 1 "187k" H 4370 3755 50  0000 L CNN
+F 2 "Resistor_SMD:R_1206_3216Metric_Pad1.42x1.75mm_HandSolder" V 4230 3800 50  0001 C CNN
+F 3 "~" H 4300 3800 50  0001 C CNN
+	1    4300 3800
+	1    0    0    -1
+$EndComp
+$Comp
+L Device:R R10
+U 1 1 5DFA8208
+P 4300 3500
+F 0 "R10" H 4370 3546 50  0000 L CNN
+F 1 "187k" H 4370 3455 50  0000 L CNN
+F 2 "Resistor_SMD:R_1206_3216Metric_Pad1.42x1.75mm_HandSolder" V 4230 3500 50  0001 C CNN
+F 3 "~" H 4300 3500 50  0001 C CNN
+	1    4300 3500
+	1    0    0    -1
+$EndComp
