File: Main.kicad_pcb (KiCad board)
At the start: 2 copper layers, 170.2 x 137.2 mm, 60 parts, among them J1 Conn_01x01_Male, J2 Conn_01x06_Male, J3 Conn_01x05_Male, J4 Conn_01x01_Male, J5 Conn_01x05_Male, J6 Conn_01x03, J7 Conn_01x03, J8 Conn_01x06, J9 Conn_01x06_Male, Q1 CSD17307Q5A, Q2 CSD17307Q5A, U1 LM4120-CustomSymbols, U2 LTC2942, U3 LM393, U4 TPS2557, U5 LM393, U6 TPS2557, U7 SN74LVC2G08

Commit message: progress
Parts:
- J3: value Conn_01x05_Male -> Conn_01x04_Male; footprint Connector_PinHeader_2.00mm:PinHeader_1x05_P2.00mm_Vertical -> Connector_PinHeader_2.00mm:PinHeader_1x04_P2.00mm_Vertical
- J9: value Conn_01x06_Male -> Conn_01x05_Male; footprint Connector_PinHeader_2.00mm:PinHeader_1x06_P2.00mm_Vertical -> Connector_PinHeader_2.00mm:PinHeader_1x05_P2.00mm_Vertical
- moved R14 87.0 mm to (151.0, 74.0), turned to 90 degrees
- moved C10 84.1 mm to (124.4, 86.7), turned to 180 degrees
- moved R19 82.5 mm to (150.9, 79.3), turned to 270 degrees
- moved R15 79.1 mm to (150.9, 68.4), turned to 90 degrees
- moved R13 76.3 mm to (138.0, 66.8), turned to 90 degrees
- moved R11 61.3 mm to (154.7, 68.4), turned to 90 degrees
- moved R17 60.2 mm to (127.8, 63.8), turned to 90 degrees
- moved R1 59.2 mm to (113.5, 69.4), turned to 270 degrees
- moved R22 57.8 mm to (134.9, 75.5), turned to 270 degrees
- moved R10 57.5 mm to (154.7, 74.0), turned to 90 degrees
- moved J9 51.2 mm to (128.9, 79.2), turned to 0 degrees
- moved R2 47.2 mm to (108.7, 69.4), turned to 270 degrees
- moved R12 46.8 mm to (138.0, 72.6), turned to 90 degrees
- moved R9 46.2 mm to (127.8, 75.1), turned to 270 degrees
- moved U7 45.9 mm to (124.8, 82.3), turned to 270 degrees
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Connections:
- J3 pad 3: BatTemp -> LowTemp
- J3 pad 4: LowTemp -> TempOK
- J9 pad 4: TempOK -> ChargeOK
- J9 pad 5: ChargeOK -> DischargeEnable
Routing:
- net 5Vref: track 7.60 -> 103.0 mm
- net ChargeOK: track 4.79 -> 35.3 mm, vias 0 -> 1
- net GNDA: track 0.00 -> 26.7 mm
- net HighTemp: track 0.95 -> 26.5 mm, vias 0 -> 1
- net PACK+: track 8.83 -> 31.9 mm
- net TempOK: track 14.5 -> 34.6 mm, vias 0 -> 4
- net DischargeOK: track 7.06 -> 23.7 mm, vias 0 -> 1
- net LowTemp: track 9.69 -> 18.1 mm
- net DischargeEnable: track 1.54 -> 9.78 mm
- net BatTemp: track 21.1 -> 28.9 mm, vias 0 -> 2
- net ChargeEnable: track 1.46 -> 7.49 mm
- net BATdiv3: track 23.7 -> 28.3 mm, vias 1 -> 2
- net 933mVref: track 12.9 -> 14.7 mm, vias 0 -> 1
- net GNDD: track 46.6 -> 47.9 mm, vias 8 -> 9
- net 1.4Vref: track 15.9 -> 16.4 mm, vias 0 -> 1
Other:
- board text removed: "5Vref"

Commit message: progress
Parts:
- moved C1 25.9 mm to (160.8, 109.3)
- moved C10 25.9 mm to (127.2, 112.5)
- moved J5 25.9 mm to (150.4, 104.0)
- moved J9 25.9 mm to (131.7, 105.0)
- moved R1 25.9 mm to (116.3, 95.1)
- moved R14 25.9 mm to (153.8, 99.8)
- moved R17 25.9 mm to (130.6, 89.6)
- moved R2 25.9 mm to (111.5, 95.1)
- moved R22 25.9 mm to (137.7, 101.2)
- moved R6 25.9 mm to (111.5, 101.4)
- moved R8 25.9 mm to (130.6, 95.0)
- moved R9 25.9 mm to (130.6, 100.9)
- moved TH1 25.9 mm to (116.3, 101.7)
- moved U3 25.9 mm to (124.3, 97.5)
- moved U5 25.9 mm to (147.3, 97.6)
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Connections:
- U7 pad 4: GNDD -> GNDA
Routing:
- net PACK+: track 31.9 -> 97.9 mm
- net ChargeEnable: track 7.49 -> 46.0 mm
- net DischargeEnable: track 9.78 -> 34.1 mm, vias 1 -> 2
- net GNDD: track 47.9 -> 67.6 mm, vias 9 -> 8
- net TempOK: track 34.6 -> 41.8 mm
- net GNDA: track 26.7 -> 31.3 mm, vias 0 -> 7
- net ChargeOK: track 35.3 -> 39.6 mm
- net MPB: track 18.6 -> 16.4 mm
- net Net-(C7-Pad1): track 12.0 -> 13.7 mm
- net Net-(R21-Pad1): track 8.65 -> 9.38 mm
- added copper zone on B.Cu, net GNDA
Other:
- board size 170.2 x 137.2 mm -> 139.7 x 81.3 mm
