File: Main.kicad_pcb (KiCad board)
At the start: 2 copper layers, 139.7 x 81.3 mm, 60 parts, among them J1 Conn_01x01_Male, J2 Conn_01x06_Male, J3 Conn_01x04_Male, J4 Conn_01x01_Male, J5 Conn_01x05_Male, J6 Conn_01x03, J7 Conn_01x03, J8 Conn_01x06, J9 Conn_01x05_Male, Q1 CSD17307Q5A, Q2 CSD17307Q5A, U1 LM4120-CustomSymbols, U2 LTC2942, U3 LM393, U4 TPS2557, U5 LM393, U6 TPS2557, U7 SN74LVC2G08

Commit message: done
Connections:
- C1 pad 2: GNDD -> GNDA
- C2 pad 2: GNDD -> GNDA
- C4 pad 2: GNDD -> GNDA
- C5 pad 2: GNDD -> GNDA
- C6 pad 2: GNDD -> GNDA
- C7 pad 2: GNDD -> GNDA
- C8 pad 2: GNDD -> GNDA
- GND1 pad 1: GNDD -> GNDA
- JP1 pad 1: GNDD -> GNDA
- Q1 pad 1: GNDD -> GNDA
- Q1 pad 2: GNDD -> GNDA
- Q1 pad 3: GNDD -> GNDA
- R20 pad 2: GNDD -> GNDA
- R21 pad 2: GNDD -> GNDA
- R3 pad 1: GNDD -> GNDA
- R4 pad 1: GNDD -> GNDA
- U1 pad 2: GNDD -> GNDA
- U2 pad 2: GNDD -> GNDA
- U4 pad 1: GNDD -> GNDA
- U6 pad 1: GNDD -> GNDA
Routing:
- net 5Vref: track 103.0 -> 2.43 mm
- net GNDD: track 67.6 -> 0.00 mm, vias 8 -> 0
- net GNDA: track 31.3 -> 78.0 mm, vias 7 -> 15
- added copper zone on F.Cu, net 5Vref
- removed copper zone on B.Cu, net GNDD
Other:
- outline, holes or cut-outs redrawn

Commit message: done
Parts:
- D1, D2: value D_Schottky -> DB2431200L; footprint Diode_SMD:D_2114_3652Metric_Castellated -> DB2431200L:DB2431200L
- moved D1 2.89 mm to (136.4, 126.7), turned to 90 degrees
- moved D2 0.36 mm to (149.4, 126.7), turned to 270 degrees
Routing:
- net Net-(C6-Pad1): track 32.6 -> 26.0 mm
Other:
- board text added: "Short Jumper"

Commit message: progress
Parts:
- moved BT1 66.2 mm to (125.0, 100.5)
- moved J2 66.2 mm to (173.8, 108.2)
- moved JP1 66.2 mm to (168.8, 90.9)
- moved C1 66.2 mm to (211.9, 67.1)
- moved C10 66.2 mm to (178.2, 70.3)
- moved C2 66.2 mm to (173.2, 102.1)
- moved C3 66.2 mm to (123.1, 78.5)
- moved C4 66.2 mm to (184.4, 93.9)
- moved C5 66.2 mm to (189.8, 93.9)
- moved C6 66.2 mm to (195.0, 93.9)
- moved C7 66.2 mm to (200.1, 93.9)
- moved C8 66.2 mm to (205.2, 93.9)
- moved C9 66.2 mm to (186.3, 53.3)
- moved CDR1 66.2 mm to (195.2, 80.6)
- moved D1 66.2 mm to (187.5, 84.6)
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Routing:
- net BatTemp: track 28.9 -> 148.4 mm, vias 2 -> 3
- net 5Vref: track 2.43 -> 74.9 mm, vias 0 -> 2
- net GNDA: track 78.0 -> 77.3 mm

Commit message: changed_footprings
Parts:
- R14: footprint Resistor_SMD:R_1206_3216Metric_Pad1.42x1.75mm_HandSolder -> Resistor_SMD:R_0805_2012Metric_Pad1.15x1.40mm_HandSolder
- R17: footprint Resistor_SMD:R_1206_3216Metric_Pad1.42x1.75mm_HandSolder -> Resistor_SMD:R_0603_1608Metric_Pad1.05x0.95mm_HandSolder
- moved R17 1.35 mm to (181.7, 48.8), turned to 180 degrees
- moved R14 0.44 mm to (204.8, 57.1)
Routing:
- net 1.4Vref: track 16.4 -> 19.1 mm
- net TempOK: track 41.8 -> 39.6 mm

Commit message: progress
Parts:
- added R24: 187k, Resistor_SMD:R_1206_3216Metric_Pad1.42x1.75mm_HandSolder, F.Cu at (208.7, 57.6)
- R1, R2, R8: value 898k -> 887k
- R10: value 332k -> 187k
- R11: value 167k -> 187k
- R12: value 1.64M -> 1.62M
- R16: value 14.7m -> 14m; footprint Resistor_SMD:R_1206_3216Metric_Pad1.42x1.75mm_HandSolder -> Resistor_SMD:R_0805_2012Metric
- U7: footprint Package_SO:SSOP-8_2.95x2.8mm_P0.65mm -> SN74LVC2G08DCTR:SN74LVC2G08DCTR
- moved R10 5.65 mm to (208.7, 63.2)
- moved R16 1.83 mm to (178.4, 102.4)
- moved U7 0.36 mm to (179.0, 65.7)
- moved R1 0.20 mm to (107.3, 86.8)
Connections:
- R10 pad 2: BATdiv3 -> Net-(R10-Pad2)
Routing:
- net GNDA: track 77.3 -> 101.1 mm
- net PACK+: track 98.0 -> 103.8 mm
- net TempOK: track 39.6 -> 44.8 mm
- net Net-(R10-Pad2): track 0.00 -> 2.65 mm
- net BAT+1: track 78.2 -> 80.5 mm, vias 1 -> 0
- net BATdiv3: track 28.3 -> 29.9 mm
- net PACK+1: track 15.6 -> 16.9 mm
- net ChargeOK: track 39.6 -> 38.8 mm
- net ChargeEnable: track 46.0 -> 45.5 mm

Commit message: gerbers
Parts:
- moved TH1 7.62 mm to (113.1, 87.8)
Routing:
- net BatTemp: track 148.4 -> 116.4 mm
Changed lines of the file:
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@@
   )
   (module Resistor_SMD:R_0402_1005Metric (layer F.Cu)
-    (at 110.085 94.8)
+    (at 113.085 87.8)
     (descr "Resistor SMD 0402 (1005 Metric), square (rectangular) end terminal, IPC_7351 nominal, (Body size source: http://www.tortai-tech.com/upload/download/2011102023233369053.pdf), generated with kicad-footprint-generator")
     (tags resistor)
@@
   (segment (start 170.2503 54.7497) (end 170.2 54.8) (width 0.25) (layer F.Cu) (net 13))
   (segment (start 172.9247 54.7497) (end 170.2503 54.7497) (width 0.25) (layer F.Cu) (net 13))
-  (segment (start 107.286 92.486) (end 109.6 94.8) (width 0.25) (layer F.Cu) (net 13))
-  (segment (start 107.286 88.1195) (end 107.286 89.714) (width 0.25) (layer F.Cu) (net 13))
-  (segment (start 107.286 89.714) (end 107.286 92.486) (width 0.25) (layer F.Cu) (net 13))
-  (via (at 107.286 89.714) (size 0.8) (drill 0.4) (layers F.Cu B.Cu) (net 13))
   (segment (start 169.800001 54.400001) (end 170.2 54.8) (width 0.25) (layer B.Cu) (net 13))
   (segment (start 135.149636 50.774999) (end 166.174999 50.774999) (width 0.25) (layer B.Cu) (net 13))
@@
   (segment (start 106.574999 83.848001) (end 106.574999 79.349636) (width 0.25) (layer B.Cu) (net 13))
   (segment (start 106.951999 84.225001) (end 106.574999 83.848001) (width 0.25) (layer B.Cu) (net 13))
-  (segment (start 122.476781 84.225001) (end 106.951999 84.225001) (width 0.25) (layer B.Cu) (net 13))
   (segment (start 166.174999 50.774999) (end 169.800001 54.400001) (width 0.25) (layer B.Cu) (net 13))
-  (segment (start 123.112279 83.589503) (end 122.476781 84.225001) (width 0.25) (layer B.Cu) (net 13))
-  (segment (start 123.112279 87.640279) (end 123.112279 83.589503) (width 0.25) (layer B.Cu) (net 13))
-  (segment (start 121.038558 89.714) (end 123.112279 87.640279) (width 0.25) (layer B.Cu) (net 13))
-  (segment (start 107.286 89.714) (end 121.038558 89.714) (width 0.25) (layer B.Cu) (net 13))
+  (segment (start 112.081 88.319) (end 112.6 87.8) (width 0.25) (layer F.Cu) (net 13))
+  (segment (start 107.315 88.319) (end 112.081 88.319) (width 0.25) (layer F.Cu) (net 13))
+  (segment (start 106.951999 84.225001) (end 109.218601 84.225001) (width 0.25) (layer B.Cu) (net 13))
+  (segment (start 109.218601 84.225001) (end 109.269401 84.225001) (width 0.25) (layer B.Cu) (net 13))
+  (segment (start 109.269401 84.225001) (end 111.7854 86.741) (width 0.25) (layer B.Cu) (net 13))
+  (segment (start 111.7854 86.741) (end 111.7854 86.741) (width 0.25) (layer B.Cu) (net 13))
+  (via (at 111.7854 86.741) (size 0.8) (drill 0.4) (layers F.Cu B.Cu) (net 13))
+  (segment (start 112.6 87.5556) (end 111.7854 86.741) (width 0.25) (layer F.Cu) (net 13))
+  (segment (start 112.6 87.8) (end 112.6 87.5556) (width 0.25) (layer F.Cu) (net 13))
   (segment (start 200.8744 61.276) (end 201.4601 61.8617) (width 0.25) (layer F.Cu) (net 14))
   (segment (start 200.8744 57.3151) (end 201.5348 57.9755) (width 0.25) (layer F.Cu) (net 14))
@@
   (segment (start 176.73 68.646502) (end 175.931999 67.848501) (width 0.25) (layer F.Cu) (net 24))
   (segment (start 176.73 70.2945) (end 176.73 68.646502) (width 0.25) (layer F.Cu) (net 24))
-  (via (at 111.5 94.7) (size 0.8) (drill 0.4) (layers F.Cu B.Cu) (net 24))
-  (segment (start 111.4 94.8) (end 111.5 94.7) (width 0.25) (layer F.Cu) (net 24))
-  (segment (start 110.57 94.8) (end 111.4 94.8) (width 0.25) (layer F.Cu) (net 24))
+  (via (at 114.5 87.7) (size 0.8) (drill 0.4) (layers F.Cu B.Cu) (net 24))
+  (segment (start 114.4 87.8) (end 114.5 87.7) (width 0.25) (layer F.Cu) (net 24))
+  (segment (start 113.57 87.8) (end 114.4 87.8) (width 0.25) (layer F.Cu) (net 24))
   (segment (start 176.5801 64.176) (end 176.5663 64.1622) (width 0.25) (layer F.Cu) (net 24))
   (segment (start 178.208 64.176) (end 176.5801 64.176) (width 0.25) (layer F.Cu) (net 24))
